File: pcb/acdc-5v/acdc-5v.kicad_pcb (KiCad board)
At the start: 2 copper layers, 72.5 x 41 mm, 12 parts, among them J1 220V, J2 5V, J3 5V, J4 GND, J5 5V

Commit message: update pcb
Other:
- board text added: "L"
- board text added: "N"
